File: examples/projtest1.kicad_pcb (KiCad board)
At the start: 2 copper layers, 6 parts, among them U1 LM555xM

Commit message: First commit
Parts:
- removed the R2 at (33.8, 17.5)
- removed R3, R4: R, Resistor_SMD:R_0612_1632Metric
- moved R2 22.7 mm to (16.8, 18.5)
- moved R1 19.9 mm to (32.8, 29.5)
- renumbered R5 to R2
Connections:
- R1 pad 1: Net-(U1-CONT) -> Net-(U1-~{RST})
- U1 pad 2: Net-(U1-TRIG) -> Net-(U1-GND)
- U1 pad 4: Net-(U1-CONT) -> Net-(U1-~{RST})
- U1 pad 5: Net-(U1-CONT) -> unconnected-(U1-CONT-Pad5)
- U1 pad 6: Net-(U1-THRES) -> unconnected-(U1-THRES-Pad6)
- U1 pad 8: Net-(U1-VCC) -> unconnected-(U1-VCC-Pad8)
Other:
- board outline added: 28 x 22.5 mm
