File: kicad_examples/example_2/projtest6.kicad_pcb (KiCad board)
At the start: 2 copper layers, 17.5 x 16.5 mm, 6 parts

Commit message: update
This commit adds a new KiCad project file with various design settings, rules, and configurations for a PCB layout.
Connections:
- net Net-(R5-Pad2) renamed GND
Changed lines of the file:
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@@
 			(layers "F.Cu" "F.Mask" "F.Paste")
 			(roundrect_rratio 0.222222)
-			(net "Net-(R5-Pad2)")
+			(net "GND")
 			(pintype "passive")
 		)
@@
 			(layers "F.Cu" "F.Mask" "F.Paste")
 			(roundrect_rratio 0.222222)
-			(net "Net-(R5-Pad2)")
+			(net "GND")
 			(pintype "passive")
 		)
